Commit message: Rebase from 'release/indigo/jackal_description'

File: urdf/accessories.urdf.xacro (robot description, xacro)
@@ -2,21 +2,24 @@
 <robot xmlns:xacro="http://www.ros.org/wiki/xacro">
   <!--
-    As you add args to this xacro, please ensure that they
-    are included with default values in each of the following
-    launch files:
+    As you add to this xacro, please be aware that both the robot and
+    simulation include it. You must retain compatibility with all of
+    the following launch files:
     jackal_viz/launch/view_model.launch
     jackal_gazebo/launch/jackal_world.launch
     jackal_base/launch/base.launch
   -->
-  <xacro:include filename="accessories/sick_lms100.urdf.xacro" />
-  <xacro:include filename="accessories/point_grey_flea.urdf.xacro" />
-  <xacro:if value="$(arg front_laser)">
-    <xacro:sick_lms100 prefix="front" />
-    <joint name="front_laser_joint" type="fixed">
-      <origin xyz="0.04 0 0.04" rpy="${PI} 0 0" />
-      <parent link="front_mount" />
-      <child link="front_laser" />
+  <xacro:include filename="accessories/sick_lms1xx.urdf.xacro" />
+  <xacro:if value="$(optenv JACKAL_LASER 0)">
+    <sick_lms1xx_mount prefix="$(optenv JACKAL_LASER_MOUNT front)"
+                       topic="$(optenv JACKAL_LASER_TOPIC scan)" />
+    <joint name="$front_laser_mount_joint" type="fixed">
+      <origin xyz="$(optenv JACKAL_LASER_OFFSET 0 0 0)"
+              rpy="$(optenv JACKAL_LASER_RPY 0 0 0)" />
+      <parent link="$(optenv JACKAL_LASER_MOUNT front)_mount" />
+      <child link="$(optenv JACKAL_LASER_MOUNT front)_laser_mount" />
     </joint>
   </xacro:if>
+  <!--
+  <xacro:include filename="accessories/point_grey_flea.urdf.xacro" />
   <xacro:if value="$(arg camera)">
     <xacro:point_grey_flea3
@@ -39,3 +42,4 @@
       />
   </xacro:if>
+  -->
 </robot>

File: urdf/accessories/sick_lms1xx.urdf.xacro (robot description, xacro)
@@ -2,5 +2,5 @@
 <!--
 Copyright (c) 2013, Goncalo Cabrita, ISR University of Coimbra
-Copyright (c) 2014, Clearpath Robotics
+Copyright (c) 2014, 2015 Clearpath Robotics
 All rights reserved.
 Redistribution and use in source and binary forms, with or without
@@ -25,5 +25,5 @@
 SOFTWARE, EVEN IF ADVISED OF THE POSSIBILITY OF SUCH DAMAGE.
 -->
-<robot  xmlns:xacro="http://ros.org/wiki/xacro" name="sick_lms100">
+<robot xmlns:xacro="http://ros.org/wiki/xacro">
   <xacro:property name="laser_x" value="0.105" />
   <xacro:property name="laser_y" value="0.102" />
@@ -39,5 +39,15 @@
     </inertial>
   </xacro:macro>
-  <xacro:macro name="sick_lms100" params="prefix">
+  <xacro:macro name="sick_lms1xx_mount" params="prefix topic">
+    <link name="${prefix}_laser_mount">
+      <visual>
+        <origin xyz="0 0 0" rpy="0 0 0" />
+        <geometry>
+          <!-- Origin of this mesh is the base of the bracket. -->
+          <mesh filename="package://jackal_description/meshes/sick-lms1xx-bracket.stl" />
+        </geometry>
+        <material name="dark_grey" />
+      </visual>
+    </link>
     <link name="${prefix}_laser">
       <xacro:box_inertial x="${laser_x}" y="${laser_y}" z="${laser_z}" mass="${laser_mass}" />
@@ -45,5 +55,6 @@
         <origin xyz="0 0 0" rpy="0 0 0" />
         <geometry>
-          <mesh filename="package://jackal_description/meshes/sick_lms100.stl" />
+          <!-- Origin of this mesh is the focal point of the LIDAR. -->
+          <mesh filename="package://jackal_description/meshes/sick-lms1xx.stl" />
         </geometry>
         <material name="light_grey" />
@@ -56,4 +67,10 @@
       </collision>
     </link>
+    <joint name="${prefix}_laser_joint" type="fixed">
+      <!-- This offset is from the base of the bracket to the LIDAR's focal point. -->
+      <origin xyz="0 0 0.149" rpy="0 0 0" />
+      <parent link="${prefix}_laser_mount" />
+      <child link="${prefix}_laser" />
+    </joint>
     <gazebo reference="${prefix}_laser">
       <material>Gazebo/Grey</material>
@@ -84,5 +101,5 @@
         </ray>
         <plugin name="gazebo_ros_laser" filename="libgazebo_ros_laser.so">
-          <topicName>scan</topicName>
+          <topicName>${topic}</topicName>
           <frameName>${prefix}_laser</frameName>
         </plugin>

File: urdf/jackal.urdf.xacro (robot description, xacro)
@@ -166,8 +166,11 @@
     <origin xyz="${mount_spacing} 0 0" />
   </joint>
-  <!-- Bring in simulation data for Gazebo -->
+  <!-- Bring in simulation data for Gazebo. -->
   <xacro:include filename="jackal.gazebo" />
-  <xacro:if value="$(arg accessories)">
-    <xacro:include filename="accessories.urdf.xacro" />
-  </xacro:if>
+  <!-- Optional standard accessories, including their simulation data. The rendering
+       of these into the final description is controlled by optenv variables, which
+       default each one to off.-->
+  <xacro:include filename="accessories.urdf.xacro" />
+  <!-- Optional custom includes. -->
+  <xacro:include filename="$(optenv JACKAL_URDF_EXTRAS empty.urdf)" />
 </robot>
