Commit message: Imported upstream version '0.5.1' of 'upstream'

File: jackal_description/urdf/accessories.urdf.xacro (robot description, xacro)
@@ -2,5 +2,5 @@
 <robot xmlns:xacro="http://www.ros.org/wiki/xacro">
   <!--
-    As you add to this xacro, please be aware that both the robot and
+    As you add to this URDF, please be aware that both the robot and
     simulation include it. You must retain compatibility with all of
     the following launch files:
@@ -9,4 +9,9 @@
     jackal_base/launch/base.launch
   -->
+  <!-- Macros to generate standoffs for offset payload mounting. -->
+  <xacro:include filename="accessories/standoffs.urdf.xacro" />
+  <!-- This optional plate mounts both the upgraded GPS and the Velodyne 3D LIDAR. -->
+  <xacro:include filename="accessories/bridge_plate.urdf.xacro" />
+  <!-- If enabled, generate the LASER payload (by default, a SICK LMS111). -->
   <xacro:include filename="accessories/sick_lms1xx.urdf.xacro" />
   <xacro:if value="$(optenv JACKAL_LASER 0)">
@@ -18,4 +23,16 @@
       <parent link="$(optenv JACKAL_LASER_MOUNT front)_mount" />
       <child link="$(optenv JACKAL_LASER_MOUNT front)_laser_mount" />
+    </joint>
+  </xacro:if>
+  <!-- If enabled, generate the upgraded Navsat payload (a Novatel Smart6). -->
+  <xacro:include filename="accessories/novatel_smart6.urdf.xacro" />
+  <xacro:if value="$(optenv JACKAL_NAVSAT 0)">
+    <bridge_plate mount="$(optenv JACKAL_NAVSAT_MOUNT rear)"
+                  height="$(optenv JACKAL_NAVSAT_HEIGHT 0.1)" />
+    <novatel_smart6 prefix="$(optenv JACKAL_NAVSAT_MOUNT rear)"/>
+    <joint name="$(optenv JACKAL_NAVSAT_MOUNT rear)_navsat_joint" type="fixed">
+      <origin xyz="0 0 0" rpy="0 0 0" />
+      <parent link="$(optenv JACKAL_NAVSAT_MOUNT rear)_bridge" />
+      <child link="$(optenv JACKAL_NAVSAT_MOUNT rear)_navsat" />
     </joint>
   </xacro:if>

Commit message: Imported upstream version '0.5.2' of 'upstream'

File: jackal_description/urdf/accessories.urdf.xacro (robot description, xacro)
@@ -14,9 +14,9 @@
   <xacro:include filename="accessories/bridge_plate.urdf.xacro" />
   <!-- If enabled, generate the LASER payload (by default, a SICK LMS111). -->
-  <xacro:include filename="accessories/sick_lms1xx.urdf.xacro" />
+  <xacro:include filename="accessories/sick_lms1xx_mount.urdf.xacro" />
   <xacro:if value="$(optenv JACKAL_LASER 0)">
     <sick_lms1xx_mount prefix="$(optenv JACKAL_LASER_MOUNT front)"
-                       topic="$(optenv JACKAL_LASER_TOPIC scan)" />
-    <joint name="$front_laser_mount_joint" type="fixed">
+                       topic="$(optenv JACKAL_LASER_TOPIC front/scan)"/>
+    <joint name="$(optenv JACKAL_LASER_MOUNT front)_laser_mount_joint" type="fixed">
       <origin xyz="$(optenv JACKAL_LASER_OFFSET 0 0 0)"
               rpy="$(optenv JACKAL_LASER_RPY 0 0 0)" />
@@ -37,26 +37,43 @@
     </joint>
   </xacro:if>
-  <!--
-  <xacro:include filename="accessories/point_grey_flea.urdf.xacro" />
-  <xacro:if value="$(arg camera)">
-    <xacro:point_grey_flea3
-      prefix="front"
-      joint_parent="front_mount"
-      joint_xyz="0.135 0 0.015"
-      joint_rpy="0 0 0"
-      camera_x="0.0754"
-      camera_y="0.029"
-      camera_z="0.035"
-      camera_mass="0.085"
-      hfov="1.0471975512"
-      width="640"
-      height="512"
-      format="R8G8B8"
-      near="0.1"
-      far="300"
-      ns="jackal"
-      frame_id="front_mount"
-      />
+  <!-- If enabled, generate the flea3 camera payload with a tilt of 30 degrees. -->
+  <xacro:include filename="accessories/camera_mount.urdf.xacro" />
+  <xacro:include filename="$(find pointgrey_camera_description)/urdf/pointgrey_flea3.urdf.xacro" />
+  <xacro:if value="$(optenv JACKAL_FLEA3 0)">
+    <camera_mount prefix="$(optenv JACKAL_FLEA_MOUNT front)"
+                       tilt="$(optenv JACKAL_FLEA_TILT 0.5236)"/>
+    <joint name="$(optenv JACKAL_FLEA3_MOUNT front)_camera_mount_joint" type="fixed">
+      <origin xyz="$(optenv JACKAL_FLEA3_OFFSET 0 0 0)"
+              rpy="$(optenv JACKAL_FLEA3_RPY 0 0 0)" />
+      <parent link="$(optenv JACKAL_FLEA_MOUNT front)_mount" />
+      <child link="$(optenv JACKAL_FLEA_MOUNT front)_camera_mount" />
+    </joint>
+    <pointgrey_flea3 frame="$(optenv JACKAL_FLEA3_MOUNT front)_camera" name="$(optenv JACKAL_FLEA_NAME front)"
+      camera_x="0.0754" camera_y="0.029" camera_z="0.035"
+      camera_mass="0.085" hfov="1.0471975512" fps="60" width="640" height="512"/>
+    <joint name="$(optenv JACKAL_FLEA3_MOUNT front)_camera_bracket_joint" type="fixed">
+      <origin xyz="0.020 0 0.0245" rpy="0 0 0" />
+      <parent link="$(optenv JACKAL_FLEA3_MOUNT front)_camera_beam" />
+      <child link="$(optenv JACKAL_FLEA3_MOUNT front)_camera" />
+    </joint>
   </xacro:if>
-  -->
+  <!-- If enabled, generate the bumblebee2 camera payload with a tilt of 0 degrees. -->
+  <xacro:include filename="accessories/camera_mount.urdf.xacro" />
+  <xacro:include filename="$(find pointgrey_camera_description)/urdf/pointgrey_bumblebee2.urdf.xacro" />
+  <xacro:if value="$(optenv JACKAL_BB2 0)">
+    <camera_mount prefix="$(optenv JACKAL_BB2_MOUNT front)"
+                        tilt="$(optenv JACKAL_BB2_TILT 0)"/>
+    <joint name="$(optenv JACKAL_BB2_MOUNT front)_camera_mount_joint" type="fixed">
+      <origin xyz="$(optenv JACKAL_BB2_OFFSET 0 0 0)"
+              rpy="$(optenv JACKAL_BB2_RPY 0 0 0)" />
+      <parent link="$(optenv JACKAL_BB2_MOUNT front)_mount" />
+      <child link="$(optenv JACKAL_BB2_MOUNT front)_camera_mount" />
+    </joint>
+    <BB2-08S2C-38 frame="$(optenv JACKAL_BB2_MOUNT front)_camera" name="$(optenv JACKAL_BB2_NAME front)" />
+    <joint name="$(optenv JACKAL_BB2_MOUNT front)_camera_bracket_joint" type="fixed">
+      <origin xyz="0.007 0 0.02450" rpy="0 0 0" />
+      <parent link="$(optenv JACKAL_BB2_MOUNT front)_camera_beam" />
+      <child link="$(optenv JACKAL_BB2_MOUNT front)_camera" />
+    </joint>
+  </xacro:if>
 </robot>

File: jackal_description/urdf/accessories/sick_lms1xx_mount.urdf.xacro (robot description, xacro)
@@ -26,18 +26,7 @@
 -->
 <robot xmlns:xacro="http://ros.org/wiki/xacro">
-  <xacro:property name="laser_x" value="0.105" />
-  <xacro:property name="laser_y" value="0.102" />
-  <xacro:property name="laser_z" value="0.152" />
-  <xacro:property name="laser_mass" value="1.1" />
-  <xacro:macro name="box_inertial" params="x y z mass">
-    <inertial>
-      <mass value="${mass}" />
-      <origin xyz="0 0 0" />
-      <inertia ixx="${0.0833333 * mass * (y*y + z*z)}" ixy="0.0" ixz="0.0"
-        iyy="${0.0833333 * mass * (x*x + z*z)}" iyz="0.0"
-        izz="${0.0833333 * mass * (x*x + y*y)}" />
-    </inertial>
-  </xacro:macro>
+  <xacro:include filename="$(find lms1xx)/urdf/sick_lms1xx.urdf.xacro" />
   <xacro:macro name="sick_lms1xx_mount" params="prefix topic">
+    <sick_lms1xx frame="${prefix}_laser" topic="${topic}" />
     <link name="${prefix}_laser_mount">
       <visual>
@@ -50,21 +39,4 @@
       </visual>
     </link>
-    <link name="${prefix}_laser">
-      <xacro:box_inertial x="${laser_x}" y="${laser_y}" z="${laser_z}" mass="${laser_mass}" />
-      <visual>
-        <origin xyz="0 0 0" rpy="0 0 0" />
-        <geometry>
-          <!-- Origin of this mesh is the focal point of the LIDAR. -->
-          <mesh filename="package://jackal_description/meshes/sick-lms1xx.stl" />
-        </geometry>
-        <material name="light_grey" />
-      </visual>
-      <collision>
-        <origin xyz="0 0 -0.05" rpy="0 0 0" />
-        <geometry>
-          <box size="${laser_x} ${laser_y} ${laser_z}" />
-        </geometry>
-      </collision>
-    </link>
     <joint name="${prefix}_laser_joint" type="fixed">
       <!-- This offset is from the base of the bracket to the LIDAR's focal point. -->
@@ -73,36 +45,6 @@
       <child link="${prefix}_laser" />
     </joint>
-    <gazebo reference="${prefix}_laser">
-      <material>Gazebo/Grey</material>
-      <turnGravityOff>true</turnGravityOff>
-      <sensor type="ray" name="${prefix}_laser">
-        <pose>0 0 0 0 0 0</pose>
-        <visualize>false</visualize>
-        <update_rate>40</update_rate>
-        <ray>
-          <scan>
-            <horizontal>
-              <samples>720</samples>
-              <resolution>1</resolution>
-              <min_angle>-1.570796</min_angle>
-              <max_angle>1.570796</max_angle>
-            </horizontal>
-          </scan>
-          <range>
-            <min>0.10</min>
-            <max>30.0</max>
-            <resolution>0.01</resolution>
-          </range>
-          <noise>
-            <type>gaussian</type>
-            <mean>0.0</mean>
-            <stddev>0.001</stddev>
-          </noise>
-        </ray>
-        <plugin name="gazebo_ros_laser" filename="libgazebo_ros_laser.so">
-          <topicName>${topic}</topicName>
-          <frameName>${prefix}_laser</frameName>
-        </plugin>
-      </sensor>
+    <gazebo reference="${prefix}_laser_mount">
+      <material>Gazebo/DarkGrey</material>
     </gazebo>
   </xacro:macro>

File: jackal_description/urdf/jackal.urdf.xacro (robot description, xacro)
@@ -33,9 +33,9 @@
       </collision>
       <inertial>
-        <origin xyz="-0.0001 0 -0.00001" rpy="0 0 0"/>
+        <origin xyz="0 0 0" rpy="0 0 0"/>
         <mass value="0.477"/>
         <inertia
-          ixx="0.0024" ixy="0" ixz="0"
-          iyy="0.0013" iyz="0"
+          ixx="0.0013" ixy="0" ixz="0"
+          iyy="0.0024" iyz="0"
           izz="0.0013"/>
       </inertial>

Commit message: Imported upstream version '0.5.3' of 'upstream'

File: jackal_description/urdf/accessories.urdf.xacro (robot description, xacro)
@@ -41,13 +41,13 @@
   <xacro:include filename="$(find pointgrey_camera_description)/urdf/pointgrey_flea3.urdf.xacro" />
   <xacro:if value="$(optenv JACKAL_FLEA3 0)">
-    <camera_mount prefix="$(optenv JACKAL_FLEA_MOUNT front)"
-                       tilt="$(optenv JACKAL_FLEA_TILT 0.5236)"/>
+    <camera_mount prefix="$(optenv JACKAL_FLEA3_MOUNT front)"
+                       tilt="$(optenv JACKAL_FLEA3_TILT 0.5236)"/>
     <joint name="$(optenv JACKAL_FLEA3_MOUNT front)_camera_mount_joint" type="fixed">
       <origin xyz="$(optenv JACKAL_FLEA3_OFFSET 0 0 0)"
               rpy="$(optenv JACKAL_FLEA3_RPY 0 0 0)" />
-      <parent link="$(optenv JACKAL_FLEA_MOUNT front)_mount" />
-      <child link="$(optenv JACKAL_FLEA_MOUNT front)_camera_mount" />
+      <parent link="$(optenv JACKAL_FLEA3_MOUNT front)_mount" />
+      <child link="$(optenv JACKAL_FLEA3_MOUNT front)_camera_mount" />
     </joint>
-    <pointgrey_flea3 frame="$(optenv JACKAL_FLEA3_MOUNT front)_camera" name="$(optenv JACKAL_FLEA_NAME front)"
+    <pointgrey_flea3 frame="$(optenv JACKAL_FLEA3_MOUNT front)_camera" name="$(optenv JACKAL_FLEA3_NAME front)"
       camera_x="0.0754" camera_y="0.029" camera_z="0.035"
       camera_mass="0.085" hfov="1.0471975512" fps="60" width="640" height="512"/>

Commit message: Imported upstream version '0.5.4' of 'upstream'

File: jackal_description/urdf/accessories.urdf.xacro (robot description, xacro)
@@ -10,9 +10,9 @@
   -->
   <!-- Macros to generate standoffs for offset payload mounting. -->
-  <xacro:include filename="accessories/standoffs.urdf.xacro" />
+  <xacro:include filename="$(find jackal_description)/urdf/accessories/standoffs.urdf.xacro" />
   <!-- This optional plate mounts both the upgraded GPS and the Velodyne 3D LIDAR. -->
-  <xacro:include filename="accessories/bridge_plate.urdf.xacro" />
+  <xacro:include filename="$(find jackal_description)/urdf/accessories/bridge_plate.urdf.xacro" />
   <!-- If enabled, generate the LASER payload (by default, a SICK LMS111). -->
-  <xacro:include filename="accessories/sick_lms1xx_mount.urdf.xacro" />
+  <xacro:include filename="$(find jackal_description)/urdf/accessories/sick_lms1xx_mount.urdf.xacro" />
   <xacro:if value="$(optenv JACKAL_LASER 0)">
     <sick_lms1xx_mount prefix="$(optenv JACKAL_LASER_MOUNT front)"
@@ -26,5 +26,5 @@
   </xacro:if>
   <!-- If enabled, generate the upgraded Navsat payload (a Novatel Smart6). -->
-  <xacro:include filename="accessories/novatel_smart6.urdf.xacro" />
+  <xacro:include filename="$(find jackal_description)/urdf/accessories/novatel_smart6.urdf.xacro" />
   <xacro:if value="$(optenv JACKAL_NAVSAT 0)">
     <bridge_plate mount="$(optenv JACKAL_NAVSAT_MOUNT rear)"
@@ -37,7 +37,8 @@
     </joint>
   </xacro:if>
+  <!-- Common camera mounts and accessory URDFs. -->
+  <xacro:include filename="$(find jackal_description)/urdf/accessories/camera_mount.urdf.xacro" />
+  <xacro:include filename="$(find pointgrey_camera_description)/urdf/pointgrey_flea3.urdf.xacro" />
   <!-- If enabled, generate the flea3 camera payload with a tilt of 30 degrees. -->
-  <xacro:include filename="accessories/camera_mount.urdf.xacro" />
-  <xacro:include filename="$(find pointgrey_camera_description)/urdf/pointgrey_flea3.urdf.xacro" />
   <xacro:if value="$(optenv JACKAL_FLEA3 0)">
     <camera_mount prefix="$(optenv JACKAL_FLEA3_MOUNT front)"
@@ -50,5 +51,5 @@
     </joint>
     <pointgrey_flea3 frame="$(optenv JACKAL_FLEA3_MOUNT front)_camera" name="$(optenv JACKAL_FLEA3_NAME front)"
-      camera_x="0.0754" camera_y="0.029" camera_z="0.035"
+      camera_x="0.0754" camera_y="0.029" camera_z="0.029"
       camera_mass="0.085" hfov="1.0471975512" fps="60" width="640" height="512"/>
     <joint name="$(optenv JACKAL_FLEA3_MOUNT front)_camera_bracket_joint" type="fixed">
@@ -58,7 +59,35 @@
     </joint>
   </xacro:if>
+  <xacro:include filename="$(find jackal_description)/urdf/accessories/stereo_camera_mount.urdf.xacro" />
+  <!-- If enabled, generates a pair of flea3 cameras for stereo vision with a tilt of 30 degrees. -->
+  <xacro:if value="$(optenv JACKAL_STEREO_FLEA3 0)">
+    <stereo_camera_mount prefix="$(optenv JACKAL_FLEA3_MOUNT front)"
+                       tilt="$(optenv JACKAL_FLEA3_TILT 0.5236)"/>
+    <joint name="$(optenv JACKAL_FLEA3_MOUNT front)_stereo_camera_mount_joint" type="fixed">
+      <origin xyz="$(optenv JACKAL_FLEA3_OFFSET 0 0 0)"
+              rpy="$(optenv JACKAL_FLEA3_RPY 0 0 0)" />
+      <parent link="$(optenv JACKAL_FLEA3_MOUNT front)_mount" />
+      <child link="$(optenv JACKAL_FLEA3_MOUNT front)_stereo_camera_mount" />
+    </joint>
+    <pointgrey_flea3 frame="$(optenv JACKAL_FLEA3_MOUNT front)_left_camera" name="$(optenv JACKAL_FLEA3_LEFT_NAME front/left)"
+      camera_x="0.0754" camera_y="0.029" camera_z="0.029"
+      camera_mass="0.085" hfov="1.0471975512" fps="60" width="640" height="512"/>
+    <joint name="$(optenv JACKAL_FLEA3_MOUNT front)_left_stereo_camera_bracket_joint" type="fixed">
+      <origin xyz="0.015 $(optenv JACKAL_STEREO_SEPERATION 0.16) 0.0599" rpy="0 0 0" />
+      <parent link="$(optenv JACKAL_FLEA3_MOUNT front)_stereo_camera_beam" />
+      <child link="$(optenv JACKAL_FLEA3_MOUNT front)_left_camera" />
+    </joint>
+    <pointgrey_flea3 frame="$(optenv JACKAL_FLEA3_MOUNT front)_right_camera" name="$(optenv JACKAL_FLEA3_RIGHT_NAME front/right)"
+      camera_x="0.0754" camera_y="0.029" camera_z="0.029"
+      camera_mass="0.085" hfov="1.0471975512" fps="60" width="640" height="512"/>
+    <joint name="$(optenv JACKAL_FLEA3_MOUNT front)_right_stereo_camera_bracket_joint" type="fixed">
+      <origin xyz="0.015 -$(optenv JACKAL_STEREO_SEPERATION 0.16) 0.0599" rpy="0 0 0" />
+      <parent link="$(optenv JACKAL_FLEA3_MOUNT front)_stereo_camera_beam" />
+      <child link="$(optenv JACKAL_FLEA3_MOUNT front)_right_camera" />
+    </joint>
+  </xacro:if>
   <!-- If enabled, generate the bumblebee2 camera payload with a tilt of 0 degrees. -->
-  <xacro:include filename="accessories/camera_mount.urdf.xacro" />
   <xacro:include filename="$(find pointgrey_camera_description)/urdf/pointgrey_bumblebee2.urdf.xacro" />
+  <!-- If enabled, generate the bumblebee2 camera payload with a tilt of 0 degrees. -->
   <xacro:if value="$(optenv JACKAL_BB2 0)">
     <camera_mount prefix="$(optenv JACKAL_BB2_MOUNT front)"

File: jackal_description/urdf/jackal.urdf.xacro (robot description, xacro)
@@ -167,10 +167,12 @@
   </joint>
   <!-- Bring in simulation data for Gazebo. -->
-  <xacro:include filename="jackal.gazebo" />
+  <xacro:include filename="$(find jackal_description)/urdf/jackal.gazebo" />
   <!-- Optional standard accessories, including their simulation data. The rendering
        of these into the final description is controlled by optenv variables, which
        default each one to off.-->
-  <xacro:include filename="accessories.urdf.xacro" />
+  <xacro:include filename="$(find jackal_description)/urdf/accessories.urdf.xacro" />
   <!-- Optional custom includes. -->
-  <xacro:include filename="$(optenv JACKAL_URDF_EXTRAS empty.urdf)" />
+  <xacro:if value="$(optenv JACKAL_URDF_EXTRAS 0)">
+    <xacro:include filename="$(env JACKAL_URDF_EXTRAS)" />
+  </xacro:if>
 </robot>
